File: ESC_V1/Hardware/esc_v1/Gate_driver_phase_U.kicad_sch (KiCad schematic)
At the start: 9 parts, among them U6 UCC27282DR

Commit message: Components roughly placed in layout
Connections:
- net GD_HB: now reaches C35.1, C36.1, U6.2 (HB)
- net GD_LO: now reaches D14.1 (K), R23.1, U6.8 (LO)
- net GD_HS: now reaches D13.1 (K), R22.1, U6.3 (HO)
Changed lines of the file:
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@@
     (stroke (width 0) (type default) (color 0 0 0 0))
+  )
+  (label "GD_HB" (at 157.48 92.71 0)
+    (effects (font (size 1.27 1.27)) (justify left bottom))
+  )
+  (label "GD_HS" (at 157.48 88.9 0)
+    (effects (font (size 1.27 1.27)) (justify left bottom))
+  )
+  (label "GD_LO" (at 157.48 109.22 0)
+    (effects (font (size 1.27 1.27)) (justify left bottom))
   )
   (hierarchical_label "HI" (shape passive) (at 116.84 96.52 180)
