File: ESC_V1/Hardware/esc_v1/Powerstage.kicad_sch (KiCad schematic)
At the start: 0 parts

Commit message: Components roughly placed in layout
Other:
- sheet three_phase_full_bridge ports: added +BATT; removed VCC
Changed lines of the file:
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@@
     (effects (font (size 1.27 1.27)) (justify right))
   )
-  (hierarchical_label "VCC" (shape passive) (at 25.4 30.48 180)
+  (hierarchical_label "+BATT" (shape passive) (at 25.4 30.48 180)
     (effects (font (size 1.27 1.27)) (justify right))
   )
@@
     (pin "1")
   )
+  (symbol (lib_id "power:+BATT") (at 110.49 54.61 0) (unit 1)
+    (in_bom yes) (on_board yes) (fields_autoplaced)
+    (property "Reference" "#PWR0104" (id 0) (at 110.49 58.42 0)
+      (effects (font (size 1.27 1.27)) hide)
+    )
+    (property "Value" "+BATT" (id 1) (at 110.49 49.53 0))
+    (property "Footprint" "" (id 2) (at 110.49 54.61 0)
+      (effects (font (size 1.27 1.27)) hide)
+    )
+    (property "Datasheet" "" (id 3) (at 110.49 54.61 0)
+      (effects (font (size 1.27 1.27)) hide)
+    )
+    (pin "1")
+  )
   (symbol (lib_id "power:+10V") (at 46.99 95.25 0) (unit 1)
     (in_bom yes) (on_board yes)
@@
     )
     (property "Datasheet" "" (id 3) (at 46.99 95.25 0)
-      (effects (font (size 1.27 1.27)) hide)
-    )
-    (pin "1")
-  )
-  (symbol (lib_id "power:VCC") (at 27.94 27.94 0) (unit 1)
-    (in_bom yes) (on_board yes) (fields_autoplaced)
-    (property "Reference" "#PWR055" (id 0) (at 27.94 31.75 0)
-      (effects (font (size 1.27 1.27)) hide)
-    )
-    (property "Value" "VCC" (id 1) (at 27.94 22.86 0))
-    (property "Footprint" "" (id 2) (at 27.94 27.94 0)
-      (effects (font (size 1.27 1.27)) hide)
-    )
-    (property "Datasheet" "" (id 3) (at 27.94 27.94 0)
       (effects (font (size 1.27 1.27)) hide)
     )
@@
     (pin "1")
   )
-  (symbol (lib_id "power:VCC") (at 110.49 54.61 0) (unit 1)
-    (in_bom yes) (on_board yes)
-    (property "Reference" "#PWR064" (id 0) (at 110.49 58.42 0)
-      (effects (font (size 1.27 1.27)) hide)
-    )
-    (property "Value" "VCC" (id 1) (at 110.49 50.8 0))
-    (property "Footprint" "" (id 2) (at 110.49 54.61 0)
-      (effects (font (size 1.27 1.27)) hide)
-    )
-    (property "Datasheet" "" (id 3) (at 110.49 54.61 0)
+  (symbol (lib_id "power:+BATT") (at 27.94 27.94 0) (unit 1)
+    (in_bom yes) (on_board yes) (fields_autoplaced)
+    (property "Reference" "#PWR0105" (id 0) (at 27.94 31.75 0)
+      (effects (font (size 1.27 1.27)) hide)
+    )
+    (property "Value" "+BATT" (id 1) (at 27.94 22.86 0))
+    (property "Footprint" "" (id 2) (at 27.94 27.94 0)
+      (effects (font (size 1.27 1.27)) hide)
+    )
+    (property "Datasheet" "" (id 3) (at 27.94 27.94 0)
       (effects (font (size 1.27 1.27)) hide)
     )
@@
       (effects (font (size 2 2)) (justify left))
     )
-    (pin "VCC" passive (at 114.3 57.15 180)
-      (effects (font (size 2 2)) (justify left))
-    )
+    (pin "+BATT" passive (at 114.3 57.15 180)
+      (effects (font (size 2 2)) (justify left))
+    )
