File: ESC_V1/Hardware/esc_v1/esc_v1.kicad_pcb (KiCad board)
At the start: 4 copper layers, 130 parts, among them J1 vcc_connector, J2 SWD_tag_connect, J3 motor_connector, J4 10118193-0001LF, Q1 IRFH7084TRPBF, Q2 IRFH7084TRPBF, Q3 IRFH7084TRPBF, Q4 IRFH7084TRPBF, Q5 IRFH7084TRPBF, Q6 IRFH7084TRPBF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

Commit message: Components roughly placed in layout
Parts:
- removed R12, R5, R6: 0R, Resistor_SMD:R_0603_1608Metric
- C46, C47, C48, C49, C50, C51, C52, C53, R28, R29, R30, R31, R32, R33, U10, U9: moved to F.Cu
- D6, D7, D8: moved to B.Cu
- moved C46 302.7 mm to (152.0, 106.5), turned to 0 degrees
- moved R28 297.6 mm to (154.5, 96.5), turned to 0 degrees
- moved C48 297.1 mm to (158.0, 104.5)
- moved R30 295.7 mm to (155.0, 105.5), turned to 90 degrees
- moved R29 293.8 mm to (158.0, 106.5)
- moved C47 291.8 mm to (152.0, 104.5), turned to 0 degrees
- moved C38 288.8 mm to (132.0, 117.0), turned to -90 degrees
- moved C49 287.2 mm to (159.0, 101.5), turned to 90 degrees
- moved U9 286.7 mm to (154.5, 101.5), turned to 0 degrees
- moved C40 285.3 mm to (134.0, 112.0), turned to 0 degrees
- moved C37 285.0 mm to (130.0, 117.0), turned to -90 degrees
- moved U7 284.7 mm to (136.0, 117.0), turned to -90 degrees
- moved C39 281.4 mm to (134.0, 110.0), turned to 0 degrees
- moved D15 277.9 mm to (141.5, 112.5), turned to 90 degrees
- moved D16 272.6 mm to (141.5, 119.5), turned to -90 degrees
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Connections:
- net Net-(C35-Pad1) renamed /Powerstage/Gate_driver_phase_U/GD_HB
- net Net-(C39-Pad1) renamed /Powerstage/Gate_driver_phase_V/GD_HB
- net Net-(C43-Pad1) renamed /Powerstage/Gate_driver_phase_W/GD_HB
- net Net-(D13-Pad1) renamed /Powerstage/Gate_driver_phase_U/GD_HS
- net Net-(D14-Pad1) renamed /Powerstage/Gate_driver_phase_U/GD_LO
- net Net-(D15-Pad1) renamed /Powerstage/Gate_driver_phase_V/GD_HS
- net Net-(D16-Pad1) renamed /Powerstage/Gate_driver_phase_V/GD_LO
- net Net-(D17-Pad1) renamed /Powerstage/Gate_driver_phase_W/GD_HS
- net Net-(D18-Pad1) renamed /Powerstage/Gate_driver_phase_W/GD_LO
- C10 pad 1: Net-(C10-Pad1) -> +10V
- C45 pad 1: VCC -> +BATT
- C6 pad 1: Net-(C6-Pad1) -> +5V
- C7 pad 1: Net-(C7-Pad1) -> +3V3
- D3 pad 1: VCC -> +BATT
- D6 pad 1: /PHASE_W -> /PHASE_V
- D7 pad 1: /PHASE_V -> /PHASE_W
- F1 pad 1: VCC -> +BATT
- J1 pad 2: VCC -> +BATT
- J3 pad 1: /PHASE_W -> /PHASE_V
- J3 pad 2: /PHASE_V -> /PHASE_W
- L1 pad 2: Net-(C10-Pad1) -> +10V
- Q1 pad 5: VCC -> +BATT
- Q1 pad 6: VCC -> +BATT
- Q1 pad 7: VCC -> +BATT
- Q1 pad 8: VCC -> +BATT
- Q3 pad 5: VCC -> +BATT
- Q3 pad 6: VCC -> +BATT
- Q3 pad 7: VCC -> +BATT
- Q3 pad 8: VCC -> +BATT
- Q5 pad 5: VCC -> +BATT
- Q5 pad 6: VCC -> +BATT
- Q5 pad 7: VCC -> +BATT
- Q5 pad 8: VCC -> +BATT
- R10 pad 1: Net-(C10-Pad1) -> +10V
- U1 pad 2: Net-(C6-Pad1) -> +5V
- U2 pad 2: Net-(C7-Pad1) -> +3V3
Other:
- rule pad_to_mask_clearance: 0.05 -> 0
