File: ESC_V1/Hardware/esc_v1/esc_v1.kicad_sch (KiCad schematic)
At the start: 19 parts, among them J1 vcc_connector, J2 SWD_tag_connect, J3 motor_connector, J4 10118193-0001LF

Commit message: Components roughly placed in layout
Connections:
- net PHASE_V: now also D6.1, J3.1 (Pin_1); no longer D7.1, J3.2 (Pin_2)
- net PHASE_W: now also D7.1, J3.2 (Pin_2); no longer D6.1, J3.1 (Pin_1)
- net VCC renamed +BATT
- no-connect marks 1 -> 2
Other:
- sheet Powerstage ports: added +BATT; removed VCC
Changed lines of the file:
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@@
   (junction (at 20.32 173.99) (diameter 0) (color 0 0 0 0)
   )
+  (no_connect (at -210.82 46.99))
   (no_connect (at 124.46 179.07))
   (bus_entry (at 40.64 82.55) (size -2.54 2.54)
@@
     (effects (font (size 1.27 1.27)) (justify left bottom))
   )
-  (label "PHASE_W" (at 68.58 138.43 180)
+  (label "PHASE_V" (at 68.58 138.43 180)
     (effects (font (size 1.27 1.27)) (justify right bottom))
   )
@@
     (effects (font (size 1.27 1.27)) (justify left bottom))
   )
-  (label "PHASE_V" (at 68.58 135.89 180)
+  (label "PHASE_W" (at 68.58 135.89 180)
     (effects (font (size 1.27 1.27)) (justify right bottom))
   )
@@
     (pin "2")
   )
+  (symbol (lib_id "power:+BATT") (at 33.02 130.81 0) (unit 1)
+    (in_bom yes) (on_board yes)
+    (property "Reference" "#PWR0103" (id 0) (at 33.02 134.62 0)
+      (effects (font (size 1.27 1.27)) hide)
+    )
+    (property "Value" "+BATT" (id 1) (at 33.02 127 0))
+    (property "Footprint" "" (id 2) (at 33.02 130.81 0)
+      (effects (font (size 1.27 1.27)) hide)
+    )
+    (property "Datasheet" "" (id 3) (at 33.02 130.81 0)
+      (effects (font (size 1.27 1.27)) hide)
+    )
+    (pin "1")
+  )
   (symbol (lib_id "power:GND") (at 212.09 148.59 0) (unit 1)
     (in_bom yes) (on_board yes)
@@
     (pin "1")
     (pin "2")
-  )
-  (symbol (lib_id "power:VCC") (at 33.02 130.81 0) (unit 1)
-    (in_bom yes) (on_board yes)
-    (property "Reference" "#PWR04" (id 0) (at 33.02 134.62 0)
-      (effects (font (size 1.27 1.27)) hide)
-    )
-    (property "Value" "VCC" (id 1) (at 33.02 127 0))
-    (property "Footprint" "" (id 2) (at 33.02 130.81 0)
-      (effects (font (size 1.27 1.27)) hide)
-    )
-    (property "Datasheet" "" (id 3) (at 33.02 130.81 0)
-      (effects (font (size 1.27 1.27)) hide)
-    )
-    (pin "1")
   )
   (symbol (lib_id "Power_Protection:PESD3V3L5UY") (at 58.42 182.88 270) (unit 4)
@@
     (pin "1")
   )
+  (symbol (lib_id "power:+BATT") (at 31.75 30.48 0) (unit 1)
+    (in_bom yes) (on_board yes) (fields_autoplaced)
+    (property "Reference" "#PWR0101" (id 0) (at 31.75 34.29 0)
+      (effects (font (size 1.27 1.27)) hide)
+    )
+    (property "Value" "+BATT" (id 1) (at 31.75 25.4 0))
+    (property "Footprint" "" (id 2) (at 31.75 30.48 0)
+      (effects (font (size 1.27 1.27)) hide)
+    )
+    (property "Datasheet" "" (id 3) (at 31.75 30.48 0)
+      (effects (font (size 1.27 1.27)) hide)
+    )
+    (pin "1")
+  )
   (symbol (lib_id "power:+5V") (at 273.05 127 0) (unit 1)
     (in_bom yes) (on_board yes) (fields_autoplaced)
@@
     )
     (property "Datasheet" "" (id 3) (at 46.99 59.69 0)
-      (effects (font (size 1.27 1.27)) hide)
-    )
-    (pin "1")
-  )
-  (symbol (lib_id "power:VCC") (at 212.09 29.21 0) (unit 1)
-    (in_bom yes) (on_board yes)
-    (property "Reference" "#PWR018" (id 0) (at 212.09 33.02 0)
-      (effects (font (size 1.27 1.27)) hide)
-    )
-    (property "Value" "VCC" (id 1) (at 212.09 25.4 0))
-    (property "Footprint" "" (id 2) (at 212.09 29.21 0)
-      (effects (font (size 1.27 1.27)) hide)
-    )
-    (property "Datasheet" "" (id 3) (at 212.09 29.21 0)
       (effects (font (size 1.27 1.27)) hide)
     )
@@
     (pin "5")
     (pin "6")
-  )
-  (symbol (lib_id "power:VCC") (at 31.75 30.48 0) (unit 1)
-    (in_bom yes) (on_board yes)
-    (property "Reference" "#PWR03" (id 0) (at 31.75 34.29 0)
-      (effects (font (size 1.27 1.27)) hide)
-    )
-    (property "Value" "VCC" (id 1) (at 31.75 26.67 0))
-    (property "Footprint" "" (id 2) (at 31.75 30.48 0)
-      (effects (font (size 1.27 1.27)) hide)
-    )
-    (property "Datasheet" "" (id 3) (at 31.75 30.48 0)
-      (effects (font (size 1.27 1.27)) hide)
-    )
-    (pin "1")
   )
   (symbol (lib_id "Device:C_Small") (at 134.62 171.45 0) (unit 1)
@@
     (pin "1")
   )
+  (symbol (lib_id "power:+BATT") (at 212.09 29.21 0) (unit 1)
+    (in_bom yes) (on_board yes) (fields_autoplaced)
+    (property "Reference" "#PWR0102" (id 0) (at 212.09 33.02 0)
+      (effects (font (size 1.27 1.27)) hide)
+    )
+    (property "Value" "+BATT" (id 1) (at 212.09 24.13 0))
+    (property "Footprint" "" (id 2) (at 212.09 29.21 0)
+      (effects (font (size 1.27 1.27)) hide)
+    )
+    (property "Datasheet" "" (id 3) (at 212.09 29.21 0)
+      (effects (font (size 1.27 1.27)) hide)
+    )
+    (pin "1")
+  )
   (symbol (lib_id "power:+3V3") (at 123.19 29.21 0) (unit 1)
     (in_bom yes) (on_board yes)
@@
       (effects (font (size 2 2)) (justify left))
     )
-    (pin "VCC" passive (at 215.9 31.75 180)
+    (pin "+BATT" passive (at 215.9 31.75 180)
       (effects (font (size 2 2)) (justify left))
     )
@@
       (reference "#PWR02") (unit 1) (value "GND") (footprint "")
     )
-    (path "/b814e4fe-9c1d-4ab7-9e82-8b90af63a125"
-      (reference "#PWR03") (unit 1) (value "VCC") (footprint "")
-    )
-    (path "/3a492d6d-fa0b-424e-b9dd-680ac0703c94"
-      (reference "#PWR04") (unit 1) (value "VCC") (footprint "")
-    )
     (path "/61ca51d1-1823-4db8-8b15-93d0887df8bc"
       (reference "#PWR05") (unit 1) (value "GND") (footprint "")
@@
       (reference "#PWR017") (unit 1) (value "+10V") (footprint "")
     )
-    (path "/803cbf80-d179-40c0-9f43-f6a2d3c07bb8"
-      (reference "#PWR018") (unit 1) (value "VCC") (footprint "")
-    )
     (path "/62464e07-b171-4ab7-820a-eef2b51df511"
       (reference "#PWR019") (unit 1) (value "GND") (footprint "")
@@
       (reference "#PWR054") (unit 1) (value "GND") (footprint "")
     )
-    (path "/691d8587-6f69-4038-a59b-9d26928d9a32/4a2d83bd-96ab-4a9c-a965-0e9c939c99c0"
-      (reference "#PWR055") (unit 1) (value "VCC") (footprint "")
-    )
     (path "/691d8587-6f69-4038-a59b-9d26928d9a32/e9f7b6f8-8e81-4a33-8690-f763412532ca"
       (reference "#PWR056") (unit 1) (value "GND") (footprint "")
@@
       (reference "#PWR063") (unit 1) (value "GND") (footprint "")
     )
-    (path "/691d8587-6f69-4038-a59b-9d26928d9a32/f7241d0d-dbbb-4a4b-90cd-67437adaeb36"
-      (reference "#PWR064") (unit 1) (value "VCC") (footprint "")
-    )
     (path "/691d8587-6f69-4038-a59b-9d26928d9a32/7b42620e-c4c9-4f2b-9f3f-c1172f0edbaf"
       (reference "#PWR065") (unit 1) (value "GND") (footprint "")
@@
       (reference "#PWR096") (unit 1) (value "GND") (footprint "")
     )
+    (path "/79f23cca-fe96-43f7-ac29-5278fe4fa098"
+      (reference "#PWR0101") (unit 1) (value "+BATT") (footprint "")
+    )
+    (path "/fb6aa6e9-055d-4aa2-b51f-d0fb01c60dd7"
+      (reference "#PWR0102") (unit 1) (value "+BATT") (footprint "")
+    )
+    (path "/28f75863-80ea-4498-ab9c-439b1882f692"
+      (reference "#PWR0103") (unit 1) (value "+BATT") (footprint "")
+    )
+    (path "/691d8587-6f69-4038-a59b-9d26928d9a32/38fc0830-4004-43f3-bc5f-fa9dd5c63ef8"
+      (reference "#PWR0104") (unit 1) (value "+BATT") (footprint "")
+    )
+    (path "/691d8587-6f69-4038-a59b-9d26928d9a32/f6954e9f-edec-451d-9be4-c0cac1c0fe1a"
+      (reference "#PWR0105") (unit 1) (value "+BATT") (footprint "")
+    )
     (path "/b987de19-cd5b-4b6a-ab5e-8f82eb9eb392"
       (reference "C1") (unit 1) (value "4.7uF") (footprint "Capacitor_SMD:C_0603_1608Metric")
@@
       (reference "R4") (unit 1) (value "1M") (footprint "Resistor_SMD:R_0603_1608Metric")
     )
-    (path "/331d98c5-7dee-4472-b71e-334dc622128d/be3a07c7-8261-4ffa-bc7e-935038f5efcd"
-      (reference "R5") (unit 1) (value "0R") (footprint "Resistor_SMD:R_0603_1608Metric")
-    )
-    (path "/331d98c5-7dee-4472-b71e-334dc622128d/37f5b2cc-8734-4229-acc1-9e75b87f8e95"
-      (reference "R6") (unit 1) (value "0R") (footprint "Resistor_SMD:R_0603_1608Metric")
-    )
     (path "/331d98c5-7dee-4472-b71e-334dc622128d/21b31269-b770-4e59-96d9-679c1df7ae41"
       (reference "R7") (unit 1) (value "4.7K") (footprint "Resistor_SMD:R_0603_1608Metric")
@@
       (reference "R11") (unit 1) (value "1.4K") (footprint "Resistor_SMD:R_0603_1608Metric")
     )
-    (path "/331d98c5-7dee-4472-b71e-334dc622128d/95f4a453-0253-4c5e-a698-cd3243616a4f"
-      (reference "R12") (unit 1) (value "0R") (footprint "Resistor_SMD:R_0603_1608Metric")
-    )
     (path "/d5927b45-4bd6-4aa1-82fe-893aae000d0e/da087297-1a3d-42b3-9858-8a11df95b7ec"
