File: Hardware/esc_v1/Gate_driver.kicad_sch (KiCad schematic)
At the start: 11 parts, among them U6 FAN7390MX

Commit message: Removed USB to serial chip and added serial connector. Finished layout, made production files and sent to production
Parts:
- D19, D20, D21: Manufacturer_Name (none) -> KYOCERA AVX; Part no DIODE SCHOTTKY 40V 2A 1206 -> SD1206S040S2R0; Producer KYOCERA AVX -> (none)
- U6: Manufacturer_Name (none) -> Fairchild; Part no (none) -> FAN7390MX
Changed lines of the file:
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@@
       (effects (font (size 1.27 1.27)) hide)
     )
-    (property "Part no" "DIODE SCHOTTKY 40V 2A 1206" (id 4) (at 152.4 106.68 90)
+    (property "Part no" "SD1206S040S2R0" (id 4) (at 152.4 106.68 90)
       (effects (font (size 1.27 1.27)) hide)
     )
-    (property "Producer" "KYOCERA AVX" (id 5) (at 152.4 106.68 90)
+    (property "Manufacturer_Name" "KYOCERA AVX" (id 5) (at 152.4 106.68 90)
       (effects (font (size 1.27 1.27)) hide)
     )
@@
       (effects (font (size 1.524 1.524)))
     )
+    (property "Part no" "FAN7390MX" (id 4) (at 119.38 81.28 0)
+      (effects (font (size 1.27 1.27)) hide)
+    )
+    (property "Manufacturer_Name" "Fairchild" (id 5) (at 119.38 81.28 0)
+      (effects (font (size 1.27 1.27)) hide)
+    )
     (pin "1")
     (pin "2")
@@
       (effects (font (size 1.27 1.27)) hide)
     )
-    (property "Part no" "DIODE SCHOTTKY 40V 2A 1206" (id 4) (at 152.4 90.17 90)
+    (property "Part no" "SD1206S040S2R0" (id 4) (at 152.4 90.17 90)
       (effects (font (size 1.27 1.27)) hide)
     )
-    (property "Producer" "KYOCERA AVX" (id 5) (at 152.4 90.17 90)
+    (property "Manufacturer_Name" "KYOCERA AVX" (id 5) (at 152.4 90.17 90)
       (effects (font (size 1.27 1.27)) hide)
     )
@@
       (effects (font (size 1.27 1.27)) hide)
     )
-    (property "Part no" "DIODE SCHOTTKY 40V 2A 1206" (id 4) (at 152.4 73.66 90)
+    (property "Part no" "SD1206S040S2R0" (id 4) (at 152.4 73.66 90)
       (effects (font (size 1.27 1.27)) hide)
     )
-    (property "Producer" "KYOCERA AVX" (id 5) (at 152.4 73.66 90)
+    (property "Manufacturer_Name" "KYOCERA AVX" (id 5) (at 152.4 73.66 90)
       (effects (font (size 1.27 1.27)) hide)
     )
