File: Hardware/esc_v1/measurements_phase_U.kicad_sch (KiCad schematic)
At the start: 8 parts, among them U9 MAX40056UAUA/V+

Commit message: changed gate driver, removed 10V buck and 5V LDO, added 5V buck. Started on Layout
Connections:
- net Ref: now reaches C48.1, C49.1, R29.1, U9.5 (REF)
Changed lines of the file:
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@@
   (title_block
     (title "Current measurement")
-    (date "2022-07-25")
+    (date "2022-08-13")
     (rev "1")
   )
@@
     (effects (font (size 2 2)) (justify left bottom))
   )
+  (label "Ref" (at 168.91 91.44 0)
+    (effects (font (size 1.27 1.27)) (justify left bottom))
+  )
   (hierarchical_label "Phase_pos" (shape passive) (at 82.55 114.3 180)

Commit message: Removed USB to serial chip and added serial connector. Finished layout, made production files and sent to production
Parts:
- R28: Manufacturer_Name (none) -> Vishay
- U9: Manufacturer_Name (none) -> Maxim Integrated; Part no (none) -> MAX40056UAUA/V+
Changed lines of the file:
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@@
+      (effects (font (size 1.27 1.27)) hide)
+    )
+    (property "Manufacturer_Name" "Vishay" (id 6) (at 111.76 114.3 90)
       (effects (font (size 1.27 1.27)) hide)
     )
@@
       (effects (font (size 1.524 1.524)) hide)
     )
+    (property "Part no" "MAX40056UAUA/V+" (id 4) (at 125.73 81.28 0)
+      (effects (font (size 1.27 1.27)) hide)
+    )
+    (property "Manufacturer_Name" "Maxim Integrated" (id 5) (at 125.73 81.28 0)
+      (effects (font (size 1.27 1.27)) hide)
+    )
     (pin "1")
