File: Hardware/esc_v1/three_phase_full_bridge.kicad_sch (KiCad schematic)
At the start: 7 parts, among them Q1 IRFH7084TRPBF, Q2 IRFH7084TRPBF, Q3 IRFH7084TRPBF, Q4 IRFH7084TRPBF, Q5 IRFH7084TRPBF, Q6 IRFH7084TRPBF

Commit message: changed gate driver, removed 10V buck and 5V LDO, added 5V buck. Started on Layout
Parts:
- removed C45: 1000uF, Capacitor_THT:CP_Radial_D10.0mm_P5.00mm, symbol Device:C_Polarized_Small
- added C40, C41: 270uF, Capacitor_SMD:CP_Elec_10x10, symbol Device:C_Polarized_Small
- added F1: 40A, Fuse:Fuse_1206_3216Metric, symbol Device:Fuse
Connections:
- net +BATT: now also F1.1; no longer Q1.5-6-7-8 (D), Q3.5-6-7-8 (D), Q5.5-6-7-8 (D)
- net GND: now also C40.2, C41.2
- new net: C40.1, C41.1, F1.2, Q1.5-6-7-8 (D), Q3.5-6-7-8 (D), Q5.5-6-7-8 (D)
Other:
- note added: "R_dson = 1.25mOhm I_max = 40A P = 0.00125*40^2 = 2W Temp increase at I_max = 70 deg C"
- note removed: "R_dson = 1.25mOhm I_max = 40A P = 0.00125*35^2 = 1.125W Temp increase = 1.125*35 = 39 deg c"
Changed lines of the file:
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@@
 (kicad_sch (version 20211123) (generator eeschema)
   (paper "A4")
+  (title_block
+    (date "2022-08-13")
+    (rev "1")
+  )
   (junction (at 151.13 127) (diameter 0) (color 0 0 0 0)
   )
   (junction (at 101.6 101.6) (diameter 0) (color 0 0 0 0)
   )
+  (junction (at 87.63 63.5) (diameter 0) (color 0 0 0 0)
+  )
+  (junction (at 83.82 72.39) (diameter 0) (color 0 0 0 0)
+  )
   (junction (at 96.52 127) (diameter 0) (color 0 0 0 0)
   )
@@
   (junction (at 151.13 101.6) (diameter 0) (color 0 0 0 0)
   )
+  (junction (at 201.93 127) (diameter 0) (color 0 0 0 0)
+  )
+  (junction (at 201.93 101.6) (diameter 0) (color 0 0 0 0)
+  )
+  (junction (at 156.21 101.6) (diameter 0) (color 0 0 0 0)
+  )
+  (junction (at 99.06 127) (diameter 0) (color 0 0 0 0)
+  )
+  (junction (at 101.6 127) (diameter 0) (color 0 0 0 0)
+  )
+  (junction (at 96.52 101.6) (diameter 0) (color 0 0 0 0)
+  )
   (junction (at 80.01 63.5) (diameter 0) (color 0 0 0 0)
   )
-  (junction (at 201.93 127) (diameter 0) (color 0 0 0 0)
-  )
-  (junction (at 201.93 101.6) (diameter 0) (color 0 0 0 0)
-  )
-  (junction (at 156.21 101.6) (diameter 0) (color 0 0 0 0)
-  )
-  (junction (at 99.06 127) (diameter 0) (color 0 0 0 0)
-  )
-  (junction (at 101.6 127) (diameter 0) (color 0 0 0 0)
-  )
-  (junction (at 96.52 101.6) (diameter 0) (color 0 0 0 0)
-  )
   (junction (at 207.01 101.6) (diameter 0) (color 0 0 0 0)
   )
@@
     (stroke (width 0) (type default) (color 0 0 0 0))
   )
-  (wire (pts (xy 96.52 63.5) (xy 80.01 63.5))
+  (wire (pts (xy 87.63 72.39) (xy 83.82 72.39))
+    (stroke (width 0) (type default) (color 0 0 0 0))
+  )
+  (wire (pts (xy 96.52 63.5) (xy 87.63 63.5))
     (stroke (width 0) (type default) (color 0 0 0 0))
   )
@@
     (stroke (width 0) (type default) (color 0 0 0 0))
   )
+  (wire (pts (xy 87.63 71.12) (xy 87.63 72.39))
+    (stroke (width 0) (type default) (color 0 0 0 0))
+  )
   (wire (pts (xy 96.52 101.6) (xy 99.06 101.6))
     (stroke (width 0) (type default) (color 0 0 0 0))
@@
     (stroke (width 0) (type default) (color 0 0 0 0))
   )
+  (wire (pts (xy 80.01 72.39) (xy 80.01 71.12))
+    (stroke (width 0) (type default) (color 0 0 0 0))
+  )
   (wire (pts (xy 153.67 127) (xy 156.21 127))
     (stroke (width 0) (type default) (color 0 0 0 0))
   )
+  (wire (pts (xy 87.63 63.5) (xy 87.63 66.04))
+    (stroke (width 0) (type default) (color 0 0 0 0))
+  )
   (wire (pts (xy 201.93 101.6) (xy 201.93 109.22))
     (stroke (width 0) (type default) (color 0 0 0 0))
@@
     (stroke (width 0) (type default) (color 0 0 0 0))
   )
+  (wire (pts (xy 87.63 63.5) (xy 80.01 63.5))
+    (stroke (width 0) (type default) (color 0 0 0 0))
+  )
   (wire (pts (xy 80.01 63.5) (xy 80.01 66.04))
     (stroke (width 0) (type default) (color 0 0 0 0))
@@
     (stroke (width 0) (type default) (color 0 0 0 0))
   )
+  (wire (pts (xy 50.8 63.5) (xy 59.69 63.5))
+    (stroke (width 0) (type default) (color 0 0 0 0))
+  )
   (wire (pts (xy 139.7 101.6) (xy 151.13 101.6))
     (stroke (width 0) (type default) (color 0 0 0 0))
@@
     (stroke (width 0) (type default) (color 0 0 0 0))
   )
-  (wire (pts (xy 80.01 63.5) (xy 76.2 63.5))
-    (stroke (width 0) (type default) (color 0 0 0 0))
-  )
   (wire (pts (xy 151.13 96.52) (xy 151.13 101.6))
     (stroke (width 0) (type default) (color 0 0 0 0))
   )
+  (wire (pts (xy 83.82 72.39) (xy 83.82 73.66))
+    (stroke (width 0) (type default) (color 0 0 0 0))
+  )
   (wire (pts (xy 76.2 127) (xy 96.52 127))
     (stroke (width 0) (type default) (color 0 0 0 0))
   )
+  (wire (pts (xy 83.82 72.39) (xy 80.01 72.39))
+    (stroke (width 0) (type default) (color 0 0 0 0))
+  )
   (wire (pts (xy 153.67 121.92) (xy 153.67 127))
     (stroke (width 0) (type default) (color 0 0 0 0))
@@
     (stroke (width 0) (type default) (color 0 0 0 0))
   )
+  (wire (pts (xy 67.31 63.5) (xy 80.01 63.5))
+    (stroke (width 0) (type default) (color 0 0 0 0))
+  )
   (wire (pts (xy 153.67 101.6) (xy 156.21 101.6))
     (stroke (width 0) (type default) (color 0 0 0 0))
@@
     (stroke (width 0) (type default) (color 0 0 0 0))
   )
-  (wire (pts (xy 80.01 71.12) (xy 80.01 73.66))
-    (stroke (width 0) (type default) (color 0 0 0 0))
-  )
-  (text "R_dson = 1.25mOhm\nI_max = 40A\nP = 0.00125*35^2 = 1.125W\nTemp increase = 1.125*35 = 39 deg c"
+  (text "R_dson = 1.25mOhm\nI_max = 40A\nP = 0.00125*40^2 = 2W\nTemp increase at I_max = 70 deg C"
     (at 138.43 71.12 0)
     (effects (font (size 1.27 1.27) bold) (justify left bottom))
@@
     (effects (font (size 1.27 1.27)) (justify right))
   )
-  (hierarchical_label "+BATT" (shape passive) (at 76.2 63.5 180)
+  (hierarchical_label "+BATT" (shape passive) (at 50.8 63.5 180)
     (effects (font (size 1.27 1.27)) (justify right))
   )
@@
   (hierarchical_label "PHASE_U" (shape passive) (at 114.3 101.6 0)
     (effects (font (size 1.27 1.27)) (justify left))
-  )
-  (symbol (lib_id "Device:C_Polarized_Small") (at 80.01 68.58 0) (unit 1)
-    (in_bom yes) (on_board yes) (fields_autoplaced)
-    (property "Reference" "C45" (id 0) (at 82.55 66.7638 0)
-      (effects (font (size 1.27 1.27)) (justify left))
-    )
-    (property "Value" "1000uF" (id 1) (at 82.55 69.3038 0)
-      (effects (font (size 1.27 1.27)) (justify left))
-    )
-    (property "Footprint" "Capacitor_THT:CP_Radial_D10.0mm_P5.00mm" (id 2) (at 80.01 68.58 0)
-      (effects (font (size 1.27 1.27)) hide)
-    )
-    (property "Datasheet" "~" (id 3) (at 80.01 68.58 0)
-      (effects (font (size 1.27 1.27)) hide)
-    )
-    (pin "1")
-    (pin "2")
   )
   (symbol (lib_id "IRFH7084TRPBF:IRFH7084TRPBF") (at 191.77 114.3 0) (unit 1)
@@
     (pin "5-6-7-8")
   )
+  (symbol (lib_id "Device:C_Polarized_Small") (at 87.63 68.58 0) (unit 1)
+    (in_bom yes) (on_board yes) (fields_autoplaced)
+    (property "Reference" "C41" (id 0) (at 90.17 66.7638 0)
+      (effects (font (size 1.27 1.27)) (justify left))
+    )
+    (property "Value" "270uF" (id 1) (at 90.17 69.3038 0)
+      (effects (font (size 1.27 1.27)) (justify left))
+    )
+    (property "Footprint" "Capacitor_SMD:CP_Elec_10x10" (id 2) (at 87.63 68.58 0)
+      (effects (font (size 1.27 1.27)) hide)
+    )
+    (property "Datasheet" "https://industrial.panasonic.com/cdbs/www-data/pdf/RDD0000/ABA0000C1221.pdf" (id 3) (at 87.63 68.58 0)
+      (effects (font (size 1.27 1.27)) hide)
+    )
+    (property "Part no" "EEH-ZA1V271V" (id 4) (at 87.63 68.58 0)
+      (effects (font (size 1.27 1.27)) hide)
+    )
+    (property "Producer" "Panasonic Electronic Components" (id 5) (at 87.63 68.58 0)
+      (effects (font (size 1.27 1.27)) hide)
+    )
+    (pin "1")
+    (pin "2")
+  )
+  (symbol (lib_id "Device:Fuse") (at 63.5 63.5 90) (unit 1)
+    (in_bom yes) (on_board yes) (fields_autoplaced)
+    (property "Reference" "F1" (id 0) (at 63.5 57.15 90))
+    (property "Value" "40A" (id 1) (at 63.5 59.69 90))
+    (property "Footprint" "Fuse:Fuse_1206_3216Metric" (id 2) (at 63.5 65.278 90)
+      (effects (font (size 1.27 1.27)) hide)
+    )
+    (property "Datasheet" "https://belfuse.com/resources/datasheets/circuitprotection/ds-CP-0685P-series.pdf" (id 3) (at 63.5 63.5 0)
+      (effects (font (size 1.27 1.27)) hide)
+    )
+    (property "Part no " "0685P9400-01" (id 4) (at 63.5 63.5 90)
+      (effects (font (size 1.27 1.27)) hide)
+    )
+    (pin "1")
+    (pin "2")
+  )
   (symbol (lib_id "power:GND") (at 96.52 133.35 0) (unit 1)
     (in_bom yes) (on_board yes) (fields_autoplaced)
@@
     (pin "5-6-7-8")
   )
+  (symbol (lib_id "Device:C_Polarized_Small") (at 80.01 68.58 0) (unit 1)
+    (in_bom yes) (on_board yes) (fields_autoplaced)
+    (property "Reference" "C40" (id 0) (at 82.55 66.7638 0)
+      (effects (font (size 1.27 1.27)) (justify left))
+    )
+    (property "Value" "270uF" (id 1) (at 82.55 69.3038 0)
+      (effects (font (size 1.27 1.27)) (justify left) hide)
+    )
+    (property "Footprint" "Capacitor_SMD:CP_Elec_10x10" (id 2) (at 80.01 68.58 0)
+      (effects (font (size 1.27 1.27)) hide)
+    )
+    (property "Datasheet" "https://industrial.panasonic.com/cdbs/www-data/pdf/RDD0000/ABA0000C1221.pdf" (id 3) (at 80.01 68.58 0)
+      (effects (font (size 1.27 1.27)) hide)
+    )
+    (property "Part no" "EEH-ZA1V271V" (id 4) (at 80.01 68.58 0)
+      (effects (font (size 1.27 1.27)) hide)
+    )
+    (property "Producer" "Panasonic Electronic Components" (id 5) (at 80.01 68.58 0)
+      (effects (font (size 1.27 1.27)) hide)
+    )
+    (pin "1")
+    (pin "2")
+  )
   (symbol (lib_id "IRFH7084TRPBF:IRFH7084TRPBF") (at 140.97 114.3 0) (unit 1)
     (in_bom yes) (on_board yes) (fields_autoplaced)
@@
     (pin "5-6-7-8")
   )
-  (symbol (lib_id "power:GND") (at 80.01 73.66 0) (unit 1)
+  (symbol (lib_id "power:GND") (at 83.82 73.66 0) (unit 1)
     (in_bom yes) (on_board yes) (fields_autoplaced)
-    (property "Reference" "#PWR087" (id 0) (at 80.01 80.01 0)
-      (effects (font (size 1.27 1.27)) hide)
-    )
-    (property "Value" "GND" (id 1) (at 80.01 78.74 0))
-    (property "Footprint" "" (id 2) (at 80.01 73.66 0)
-      (effects (font (size 1.27 1.27)) hide)
-    )
-    (property "Datasheet" "" (id 3) (at 80.01 73.66 0)
-      (effects (font (size 1.27 1.27)) hide)
-    )
+    (property "Reference" "#PWR087" (id 0) (at 83.82 80.01 0)
+      (effects (font (size 1.27 1.27)) hide)
+    )
+    (property "Value" "GND" (id 1) (at 83.82 78.74 0))
+    (property "Footprint" "" (id 2) (at 83.82 73.66 0)
+      (effects (font (size 1.27 1.27)) hide)
+    )
+    (property "Datasheet" "" (id 3) (at 83.82 73.66 0)
+      (effects (font (size 1.27 1.27)) hide)
+    )

Commit message: Changed to 6 layer pcb, increased space by 10mm, redid gate driver traces and power planes
Parts:
- added TP10, TP11, TP12, TP7, TP8, TP9: TestPoint, TestPoint:TestPoint_Pad_D2.0mm, symbol Connector:TestPoint
Connections:
- net H_U: now also TP7.1
- net H_V: now also TP9.1
- net H_W: now also TP11.1
- net L_U: now also TP8.1
- net L_V: now also TP10.1
- net L_W: now also TP12.1
Changed lines of the file:
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@@
     (rev "1")
   )
+  (junction (at 191.77 88.9) (diameter 0) (color 0 0 0 0)
+  )
   (junction (at 151.13 127) (diameter 0) (color 0 0 0 0)
   )
@@
   (junction (at 101.6 127) (diameter 0) (color 0 0 0 0)
   )
+  (junction (at 78.74 114.3) (diameter 0) (color 0 0 0 0)
+  )
   (junction (at 96.52 101.6) (diameter 0) (color 0 0 0 0)
   )
+  (junction (at 191.77 114.3) (diameter 0) (color 0 0 0 0)
+  )
   (junction (at 80.01 63.5) (diameter 0) (color 0 0 0 0)
   )
+  (junction (at 140.97 114.3) (diameter 0) (color 0 0 0 0)
+  )
   (junction (at 207.01 101.6) (diameter 0) (color 0 0 0 0)
   )
@@
   (junction (at 151.13 76.2) (diameter 0) (color 0 0 0 0)
   )
+  (junction (at 140.97 88.9) (diameter 0) (color 0 0 0 0)
+  )
+  (junction (at 78.74 88.9) (diameter 0) (color 0 0 0 0)
+  )
   (junction (at 156.21 127) (diameter 0) (color 0 0 0 0)
   )
@@
     (stroke (width 0) (type default) (color 0 0 0 0))
   )
-  (wire (pts (xy 139.7 114.3) (xy 143.51 114.3))
+  (wire (pts (xy 140.97 88.9) (xy 143.51 88.9))
+    (stroke (width 0) (type default) (color 0 0 0 0))
+  )
+  (wire (pts (xy 191.77 114.3) (xy 194.31 114.3))
+    (stroke (width 0) (type default) (color 0 0 0 0))
+  )
+  (wire (pts (xy 139.7 114.3) (xy 140.97 114.3))
     (stroke (width 0) (type default) (color 0 0 0 0))
   )
@@
     (stroke (width 0) (type default) (color 0 0 0 0))
   )
+  (wire (pts (xy 140.97 86.36) (xy 140.97 88.9))
+    (stroke (width 0) (type default) (color 0 0 0 0))
+  )
   (wire (pts (xy 96.52 101.6) (xy 99.06 101.6))
     (stroke (width 0) (type default) (color 0 0 0 0))
   )
+  (wire (pts (xy 191.77 86.36) (xy 191.77 88.9))
+    (stroke (width 0) (type default) (color 0 0 0 0))
+  )
   (wire (pts (xy 99.06 101.6) (xy 101.6 101.6))
     (stroke (width 0) (type default) (color 0 0 0 0))
@@
     (stroke (width 0) (type default) (color 0 0 0 0))
   )
+  (wire (pts (xy 78.74 111.76) (xy 78.74 114.3))
+    (stroke (width 0) (type default) (color 0 0 0 0))
+  )
   (wire (pts (xy 201.93 101.6) (xy 201.93 109.22))
     (stroke (width 0) (type default) (color 0 0 0 0))
@@
     (stroke (width 0) (type default) (color 0 0 0 0))
   )
+  (wire (pts (xy 78.74 86.36) (xy 78.74 88.9))
+    (stroke (width 0) (type default) (color 0 0 0 0))
+  )
   (wire (pts (xy 151.13 101.6) (xy 151.13 109.22))
     (stroke (width 0) (type default) (color 0 0 0 0))
@@
     (stroke (width 0) (type default) (color 0 0 0 0))
   )
-  (wire (pts (xy 190.5 114.3) (xy 194.31 114.3))
+  (wire (pts (xy 190.5 114.3) (xy 191.77 114.3))
+    (stroke (width 0) (type default) (color 0 0 0 0))
+  )
+  (wire (pts (xy 191.77 111.76) (xy 191.77 114.3))
     (stroke (width 0) (type default) (color 0 0 0 0))
   )
@@
     (stroke (width 0) (type default) (color 0 0 0 0))
   )
-  (wire (pts (xy 190.5 88.9) (xy 194.31 88.9))
+  (wire (pts (xy 190.5 88.9) (xy 191.77 88.9))
     (stroke (width 0) (type default) (color 0 0 0 0))
   )
@@
     (stroke (width 0) (type default) (color 0 0 0 0))
   )
-  (wire (pts (xy 76.2 88.9) (xy 88.9 88.9))
+  (wire (pts (xy 76.2 88.9) (xy 78.74 88.9))
     (stroke (width 0) (type default) (color 0 0 0 0))
   )
@@
     (stroke (width 0) (type default) (color 0 0 0 0))
   )
+  (wire (pts (xy 78.74 88.9) (xy 88.9 88.9))
+    (stroke (width 0) (type default) (color 0 0 0 0))
+  )
   (wire (pts (xy 207.01 127) (xy 204.47 127))
     (stroke (width 0) (type default) (color 0 0 0 0))
@@
     (stroke (width 0) (type default) (color 0 0 0 0))
   )
+  (wire (pts (xy 78.74 114.3) (xy 88.9 114.3))
+    (stroke (width 0) (type default) (color 0 0 0 0))
+  )
   (wire (pts (xy 50.8 63.5) (xy 59.69 63.5))
     (stroke (width 0) (type default) (color 0 0 0 0))
@@
     (stroke (width 0) (type default) (color 0 0 0 0))
   )
+  (wire (pts (xy 191.77 88.9) (xy 194.31 88.9))
+    (stroke (width 0) (type default) (color 0 0 0 0))
+  )
   (wire (pts (xy 190.5 101.6) (xy 201.93 101.6))
     (stroke (width 0) (type default) (color 0 0 0 0))
@@
     (stroke (width 0) (type default) (color 0 0 0 0))
   )
-  (wire (pts (xy 139.7 88.9) (xy 143.51 88.9))
+  (wire (pts (xy 140.97 114.3) (xy 143.51 114.3))
+    (stroke (width 0) (type default) (color 0 0 0 0))
+  )
+  (wire (pts (xy 139.7 88.9) (xy 140.97 88.9))
     (stroke (width 0) (type default) (color 0 0 0 0))
   )
@@
     (stroke (width 0) (type default) (color 0 0 0 0))
   )
+  (wire (pts (xy 140.97 111.76) (xy 140.97 114.3))
+    (stroke (width 0) (type default) (color 0 0 0 0))
+  )
   (wire (pts (xy 96.52 76.2) (xy 96.52 83.82))
     (stroke (width 0) (type default) (color 0 0 0 0))
   )
-  (wire (pts (xy 76.2 114.3) (xy 88.9 114.3))
+  (wire (pts (xy 76.2 114.3) (xy 78.74 114.3))
     (stroke (width 0) (type default) (color 0 0 0 0))
   )
@@
     (pin "5-6-7-8")
   )
+  (symbol (lib_id "Connector:TestPoint") (at 191.77 111.76 0) (unit 1)
+    (in_bom yes) (on_board yes)
+    (property "Reference" "TP12" (id 0) (at 194.31 109.22 90))
+    (property "Value" "TestPoint" (id 1) (at 194.31 109.7279 0)
+      (effects (font (size 1.27 1.27)) (justify left) hide)
+    )
+    (property "Footprint" "TestPoint:TestPoint_Pad_D2.0mm" (id 2) (at 196.85 111.76 0)
+      (effects (font (size 1.27 1.27)) hide)
+    )
+    (property "Datasheet" "~" (id 3) (at 196.85 111.76 0)
+      (effects (font (size 1.27 1.27)) hide)
+    )
+    (pin "1")
+  )
   (symbol (lib_id "IRFH7084TRPBF:IRFH7084TRPBF") (at 140.97 88.9 0) (unit 1)
     (in_bom yes) (on_board yes) (fields_autoplaced)
@@
     (pin "1")
     (pin "2")
+  )
+  (symbol (lib_id "Connector:TestPoint") (at 78.74 111.76 0) (unit 1)
+    (in_bom yes) (on_board yes)
+    (property "Reference" "TP8" (id 0) (at 81.28 109.22 90))
+    (property "Value" "TestPoint" (id 1) (at 81.28 109.7279 0)
+      (effects (font (size 1.27 1.27)) (justify left) hide)
+    )
+    (property "Footprint" "TestPoint:TestPoint_Pad_D2.0mm" (id 2) (at 83.82 111.76 0)
+      (effects (font (size 1.27 1.27)) hide)
+    )
+    (property "Datasheet" "~" (id 3) (at 83.82 111.76 0)
+      (effects (font (size 1.27 1.27)) hide)
+    )
+    (pin "1")
   )
   (symbol (lib_id "Device:Fuse") (at 63.5 63.5 90) (unit 1)
@@
     (pin "5-6-7-8")
   )
+  (symbol (lib_id "Connector:TestPoint") (at 191.77 86.36 0) (unit 1)
+    (in_bom yes) (on_board yes)
+    (property "Reference" "TP11" (id 0) (at 194.31 83.82 90))
+    (property "Value" "TestPoint" (id 1) (at 194.31 84.3279 0)
+      (effects (font (size 1.27 1.27)) (justify left) hide)
+    )
+    (property "Footprint" "TestPoint:TestPoint_Pad_D2.0mm" (id 2) (at 196.85 86.36 0)
+      (effects (font (size 1.27 1.27)) hide)
+    )
+    (property "Datasheet" "~" (id 3) (at 196.85 86.36 0)
+      (effects (font (size 1.27 1.27)) hide)
+    )
+    (pin "1")
+  )
   (symbol (lib_id "Device:C_Polarized_Small") (at 80.01 68.58 0) (unit 1)
     (in_bom yes) (on_board yes) (fields_autoplaced)
@@
     (pin "2")
   )
+  (symbol (lib_id "Connector:TestPoint") (at 140.97 111.76 0) (unit 1)
+    (in_bom yes) (on_board yes)
+    (property "Reference" "TP10" (id 0) (at 143.51 109.22 90))
+    (property "Value" "TestPoint" (id 1) (at 143.51 109.7279 0)
+      (effects (font (size 1.27 1.27)) (justify left) hide)
+    )
+    (property "Footprint" "TestPoint:TestPoint_Pad_D2.0mm" (id 2) (at 146.05 111.76 0)
+      (effects (font (size 1.27 1.27)) hide)
+    )
+    (property "Datasheet" "~" (id 3) (at 146.05 111.76 0)
+      (effects (font (size 1.27 1.27)) hide)
+    )
+    (pin "1")
+  )
+  (symbol (lib_id "Connector:TestPoint") (at 140.97 86.36 0) (unit 1)
+    (in_bom yes) (on_board yes)
+    (property "Reference" "TP9" (id 0) (at 143.51 83.82 90))
+    (property "Value" "TestPoint" (id 1) (at 143.51 84.3279 0)
+      (effects (font (size 1.27 1.27)) (justify left) hide)
+    )
+    (property "Footprint" "TestPoint:TestPoint_Pad_D2.0mm" (id 2) (at 146.05 86.36 0)
+      (effects (font (size 1.27 1.27)) hide)
+    )
+    (property "Datasheet" "~" (id 3) (at 146.05 86.36 0)
+      (effects (font (size 1.27 1.27)) hide)
+    )
+    (pin "1")
+  )
+  (symbol (lib_id "Connector:TestPoint") (at 78.74 86.36 0) (unit 1)
+    (in_bom yes) (on_board yes)
+    (property "Reference" "TP7" (id 0) (at 81.28 83.82 90))
+    (property "Value" "TestPoint" (id 1) (at 81.28 84.3279 0)
+      (effects (font (size 1.27 1.27)) (justify left) hide)
+    )
+    (property "Footprint" "TestPoint:TestPoint_Pad_D2.0mm" (id 2) (at 83.82 86.36 0)
+      (effects (font (size 1.27 1.27)) hide)
+    )
+    (property "Datasheet" "~" (id 3) (at 83.82 86.36 0)
+      (effects (font (size 1.27 1.27)) hide)
+    )
+    (pin "1")
+  )
   (symbol (lib_id "IRFH7084TRPBF:IRFH7084TRPBF") (at 140.97 114.3 0) (unit 1)
