File: Hardware/esc_v1/three_phase_full_bridge.kicad_sch (KiCad schematic)
At the start: 15 parts, among them Q1 IRFH7084TRPBF, Q2 IRFH7084TRPBF, Q3 IRFH7084TRPBF, Q4 IRFH7084TRPBF, Q5 IRFH7084TRPBF, Q6 IRFH7084TRPBF

Commit message: Removed USB to serial chip and added serial connector. Finished layout, made production files and sent to production
Parts:
- C40, C41: Manufacturer_Name (none) -> Panasonic Electronic Components; Producer Panasonic Electronic Components -> (none)
- F1: Manufacturer_Name (none) -> Belfuse; Part no (none) -> 0685P9400-01; Part no  0685P9400-01 -> (none)
- Q1, Q2, Q3, Q4, Q5, Q6: Manufacturer_Name (none) -> Infineon; Part no (none) -> IRFH7084TRPBF; manufacturer Infineon -> (none)
Changed lines of the file:
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@@
       (effects (font (size 1.27 1.27)) (justify left) hide)
     )
-    (property "manufacturer" "Infineon" (id 22) (at 191.77 50.8 0)
+    (property "Manufacturer_Name" "Infineon" (id 22) (at 191.77 50.8 0)
       (effects (font (size 1.27 1.27)) (justify left) hide)
     )
@@
     (property "turn on delay time" "16ns" (id 40) (at 191.77 5.08 0)
       (effects (font (size 1.27 1.27)) (justify left) hide)
+    )
+    (property "Part no" "IRFH7084TRPBF" (id 41) (at 191.77 114.3 0)
+      (effects (font (size 1.27 1.27)) hide)
     )
     (pin "1")
@@
       (effects (font (size 1.27 1.27)) (justify left) hide)
     )
-    (property "manufacturer" "Infineon" (id 22) (at 86.36 25.4 0)
+    (property "Manufacturer_Name" "Infineon" (id 22) (at 86.36 25.4 0)
       (effects (font (size 1.27 1.27)) (justify left) hide)
     )
@@
     (property "turn on delay time" "16ns" (id 40) (at 86.36 -20.32 0)
       (effects (font (size 1.27 1.27)) (justify left) hide)
+    )
+    (property "Part no" "IRFH7084TRPBF" (id 41) (at 86.36 88.9 0)
+      (effects (font (size 1.27 1.27)) hide)
     )
     (pin "1")
@@
       (effects (font (size 1.27 1.27)) (justify left) hide)
     )
-    (property "manufacturer" "Infineon" (id 22) (at 140.97 25.4 0)
+    (property "Manufacturer_Name" "Infineon" (id 22) (at 140.97 25.4 0)
       (effects (font (size 1.27 1.27)) (justify left) hide)
     )
@@
     (property "turn on delay time" "16ns" (id 40) (at 140.97 -20.32 0)
       (effects (font (size 1.27 1.27)) (justify left) hide)
+    )
+    (property "Part no" "IRFH7084TRPBF" (id 41) (at 140.97 88.9 0)
+      (effects (font (size 1.27 1.27)) hide)
     )
     (pin "1")
@@
       (effects (font (size 1.27 1.27)) (justify left) hide)
     )
-    (property "manufacturer" "Infineon" (id 22) (at 86.36 50.8 0)
+    (property "Manufacturer_Name" "Infineon" (id 22) (at 86.36 50.8 0)
       (effects (font (size 1.27 1.27)) (justify left) hide)
     )
@@
     (property "turn on delay time" "16ns" (id 40) (at 86.36 5.08 0)
       (effects (font (size 1.27 1.27)) (justify left) hide)
+    )
+    (property "Part no" "IRFH7084TRPBF" (id 41) (at 86.36 114.3 0)
+      (effects (font (size 1.27 1.27)) hide)
     )
     (pin "1")
@@
       (effects (font (size 1.27 1.27)) hide)
     )
-    (property "Producer" "Panasonic Electronic Components" (id 5) (at 87.63 68.58 0)
+    (property "Manufacturer_Name" "Panasonic Electronic Components" (id 5) (at 87.63 68.58 0)
       (effects (font (size 1.27 1.27)) hide)
     )
@@
       (effects (font (size 1.27 1.27)) hide)
     )
-    (property "Part no " "0685P9400-01" (id 4) (at 63.5 63.5 90)
+    (property "Part no" "0685P9400-01" (id 4) (at 63.5 63.5 90)
+      (effects (font (size 1.27 1.27)) hide)
+    )
+    (property "Manufacturer_Name" "Belfuse" (id 5) (at 63.5 63.5 90)
       (effects (font (size 1.27 1.27)) hide)
     )
@@
       (effects (font (size 1.27 1.27)) (justify left) hide)
     )
-    (property "manufacturer" "Infineon" (id 22) (at 191.77 25.4 0)
+    (property "Manufacturer_Name" "Infineon" (id 22) (at 191.77 25.4 0)
       (effects (font (size 1.27 1.27)) (justify left) hide)
     )
@@
     (property "turn on delay time" "16ns" (id 40) (at 191.77 -20.32 0)
       (effects (font (size 1.27 1.27)) (justify left) hide)
+    )
+    (property "Part no" "IRFH7084TRPBF" (id 41) (at 191.77 88.9 0)
+      (effects (font (size 1.27 1.27)) hide)
     )
     (pin "1")
@@
       (effects (font (size 1.27 1.27)) hide)
     )
-    (property "Producer" "Panasonic Electronic Components" (id 5) (at 80.01 68.58 0)
+    (property "Manufacturer_Name" "Panasonic Electronic Components" (id 5) (at 80.01 68.58 0)
       (effects (font (size 1.27 1.27)) hide)
     )
@@
       (effects (font (size 1.27 1.27)) (justify left) hide)
     )
-    (property "manufacturer" "Infineon" (id 22) (at 140.97 50.8 0)
+    (property "Manufacturer_Name" "Infineon" (id 22) (at 140.97 50.8 0)
       (effects (font (size 1.27 1.27)) (justify left) hide)
     )
@@
       (effects (font (size 1.27 1.27)) (justify left) hide)
     )
-    (pin "1")
+    (property "Part no" "IRFH7084TRPBF" (id 41) (at 140.97 114.3 0)
+      (effects (font (size 1.27 1.27)) hide)
+    )
+    (pin "1")
